Commit message: Initial commit

File: resources/robots/balio/urdf/balio_issac_gym_new.urdf (robot description, URDF)
Before this commit: robot wl, 7 links, 6 joints
Links:
- link l_wheel_Link: geometry collision mesh filename=../meshes/wheel1.STL; visual mesh filename=../meshes/wheel1.STL
- link lf0_Link: geometry collision mesh filename=../meshes/leg2_up.STL; visual mesh filename=../meshes/leg2_up.STL
- link lf1_Link: geometry collision mesh filename=../meshes/leg2_down.STL; visual mesh filename=../meshes/leg2_down.STL
- link r_wheel_Link: geometry collision mesh filename=../meshes/wheel1.STL; visual mesh filename=../meshes/wheel1.STL
- link rf0_Link: geometry collision mesh filename=../meshes/leg2_up.STL; visual mesh filename=../meshes/leg2_up.STL
- link rf1_Link: geometry collision mesh filename=../meshes/leg2_down.STL; visual mesh filename=../meshes/leg2_down.STL
